Commit message: Update and rename piatek.urdf to exercici51.urdf

File: urdf/exercici51.urdf (robot description, URDF)
Before this commit: robot piatek, 2 links, 0 joints
Links:
- link motor_camera_link: geometry visual mesh filename=package://Exercici5.1/urdf/meshes/Final_design.stl scale=0.001 0.001 0.001
